File: hardware/kicad/TES_Controller.kicad_pcb (KiCad board)
At the start: 2 copper layers, 64.1 x 89.3 mm, 79 parts

Commit message: Make the board and schematic agree on one footprint library
The board's footprints pointed at a library called TES_Contro-easyedapro
that does not exist, while the schematic assigned TES:. That is not just a
warning — the first time anyone runs "Update PCB from Schematic" in the GUI,
all 73 footprints get swapped and the routing goes with them.

Fixing it turned up something I had got wrong earlier. easyeda2kicad works
from LCSC part numbers, so it skips generic parts, and I concluded the 5 mm
LED, the 2.54 mm headers and the solder jumper had no footprints and drew
them myself. The EasyEDA Pro project zip has them all along; they came in
with the board import. The two versions differ — the LED's pin 1 is on the
opposite side and the drill is 1.00 mm rather than 0.90 — and the imported
ones are what V1.1 and V1.2 were actually built and soldered with, so those
win. tools/pcb_export_fp.py writes the board's footprints out to TES.pretty,
carrying over the 3D model references the board copies lack, and the symbols
and the footprint generator now point at them.

Dangling copper is gone too: 8 tracks, 1 via and 2 vias drilled straight
through U10's through-hole pad, the last from routing that places a via at
the start of a path when that start is already a plated hole. It took four
passes, since removing one layer of stubs exposes the next.

That clean-up also cost a connection on the first attempt. Matching the DRC
report by coordinate alone deletes every track sharing that endpoint, not
the dangling one; the report's length field distinguishes them.

The 60 remaining library mismatches are text-position differences between
rotated instances and the single canonical copy — one exported footprint
cannot match 19 differently-rotated R0603 placements. Warning only, and it
does not affect what gets fabricated.

DRC: zero errors, zero unconnected, 174 warnings. ERC clean, netlist still
226 connections with zero difference.

Co-Authored-By: Claude Opus 5 <noreply@anthropic.co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
Parts:
- BOOT1, EN1: footprint TES_Contro-easyedapro:SW-SMD_L3.9-W3.0-P4.45 -> TES:SW-SMD_L3.9-W3.0-P4.45
- C1, C10, C16, C17, C9: footprint TES_Contro-easyedapro:C1206 -> TES:C1206
- C11, C12, C13, C14, C15, C2, C20, C28, C29, C3, C4, C7, C8: footprint TES_Contro-easyedapro:C0603 -> TES:C0603
- CN1: footprint TES_Contro-easyedapro:CONN-TH_B2PS-VH-LF-SN -> TES:CONN-TH_B2PS-VH-LF-SN
- CN2: footprint TES_Contro-easyedapro:CONN-TH_S4B-XH-A-LF-SN -> TES:CONN-TH_S4B-XH-A-LF-SN
- CN3, CN5, CN6: footprint TES_Contro-easyedapro:CONN-TH_2P-P3.50_DG381-3.5-02P-14-00A -> TES:CONN-TH_2P-P3.50_DG381-3.5-02P-14-00A
- D1, D4: footprint TES_Contro-easyedapro:SMA_L4.2-W2.6-LS5.0-RD_1 -> TES:SMA_L4.2-W2.6-LS5.0-RD_1
- D10, D9: footprint SMB_L4.6-W3.6-LS5.3-RD -> TES:SMB_L4.6-W3.6-LS5.3-RD
- D3: footprint TES_Contro-easyedapro:SMB_L4.6-W3.6-LS5.3-RD -> TES:SMB_L4.6-W3.6-LS5.3-RD
- D5: footprint TES_Contro-easyedapro:SOT-23-6_L2.9-W1.6-P0.95-LS2.8-BL -> TES:SOT-23-6_L2.9-W1.6-P0.95-LS2.8-BL
- D6, D7, D8: footprint TES_Contro-easyedapro:LED-TH_BD5.8-P2.54-FD -> TES:LED-TH_BD5.8-P2.54-FD
- EMERGENCY1, SETTING1, START1, STOP1: footprint TES_Contro-easyedapro:SW-SMD_4P-L5.1-W5.1-P3.70-LS6.5-TL_H1.5 -> TES:SW-SMD_4P-L5.1-W5.1-P3.70-LS6.5-TL_H1.5
- H1: footprint TES_Contro-easyedapro:HDR-TH_4P-P2.54-V-F -> TES:HDR-TH_4P-P2.54-V-F
- H2: footprint TES_Contro-easyedapro:HDR-TH_3P-P2.54-V-F -> TES:HDR-TH_3P-P2.54-V-F
- Q1, Q2, Q3: footprint TES_Contro-easyedapro:SOT-23-3_L2.9-W1.3-P1.90-LS2.4-BR -> TES:SOT-23-3_L2.9-W1.3-P1.90-LS2.4-BR
- Q4: footprint TES_Contro-easyedapro:SOT-23_L2.9-W1.3-P1.90-LS2.4-BR -> TES:SOT-23_L2.9-W1.3-P1.90-LS2.4-BR
- R1, R10, R11, R12, R13, R14, R16, R17, R19, R20, R21, R26, R28, R29, R30, R31, R32, R5, R6: footprint TES_Contro-easyedapro:R0603 -> TES:R0603
- R2, R3: footprint TES_Contro-easyedapro:R0402 -> TES:R0402
- R8: footprint TES_Contro-easyedapro:R1206 -> TES:R1206
- R9: footprint TES_Contro-easyedapro:R1210 -> TES:R1210
- SB1: footprint TES_Contro-easyedapro:PAD-JUMPER-2-NC_BY_PASTE_YES_SILK -> TES:PAD-JUMPER-2-NC_BY_PASTE_YES_SILK
- U1: footprint TES_Contro-easyedapro:WIRELM-SMD_ESP32-S3-WROOM-1 -> TES:WIRELM-SMD_ESP32-S3-WROOM-1
- U10: footprint TES_Contro-easyedapro:CONN-TH_DEGSON_DG301-5.0-02P -> TES:CONN-TH_DEGSON_DG301-5.0-02P
- U12: footprint TES_Contro-easyedapro:SOIC-8_L4.9-W3.9-P1.27-LS6.0-BL -> TES:SOIC-8_L4.9-W3.9-P1.27-LS6.0-BL
- U5: footprint TES_Contro-easyedapro:MSOP-10_L3.0-W3.0-P0.50-LS5.0-BL -> TES:MSOP-10_L3.0-W3.0-P0.50-LS5.0-BL
- U6: footprint TES_Contro-easyedapro:SOT-223-3_L6.5-W3.4-P2.30-LS7.0-BR -> TES:SOT-223-3_L6.5-W3.4-P2.30-LS7.0-BR
- U8: footprint TES_Contro-easyedapro:USIP-10_L3.8-W3.0-TL_TI_SIL -> TES:USIP-10_L3.8-W3.0-TL_TI_SIL
- USB1: footprint TES_Contro-easyedapro:USB-C-SMD_TYPE-C16PIN -> TES:USB-C-SMD_TYPE-C16PIN
- W1: footprint Pad_e146 -> TES:SOLDERPAD-TH_3.0X1.5
- W2: footprint Pad_e128 -> TES:SOLDERPAD-TH_3.0X1.5
- W3: footprint Pad_e150 -> TES:SOLDERPAD-TH_3.0X1.5
- W4: footprint Pad_e125 -> TES:SOLDERPAD-TH_3.0X1.5
Routing:
- net SDA: track 48.1 -> 38.8 mm
- net VDD33: track 95.6 -> 86.7 mm
- net 5V: track 62.7 -> 61.3 mm, vias 10 -> 9
- net UD-: track 8.42 -> 7.26 mm
- net UD+: track 8.06 -> 6.91 mm
- net USB_DN_ESD: track 43.3 -> 42.2 mm
- net 120V: vias 5 -> 4

Commit message: Split R10 so no resistor sits above its rated voltage
R10 is a single 0603 carrying the top half of the 120 V sense divider. A
0603's rated working voltage is 75 V; at 120 V input it sees 116 V, half
again over the limit. This is not thin margin, it is continuous operation
out of spec, and the failure mode is quiet: the resistor drifts upward,
which lowers the divided voltage, so the charger reads the pack as lower
than it is and reports that to the vehicle.

118k + 115k + 115k comes to exactly 348k, so the divider ratio is unchanged
and AIN0 still sits at 4.0000 V at 120 V input — no firmware constant moves.
All three are E96 values. Each drops 38-39 V, giving 1.9x margin on the 75 V
rating, and dissipates 13 mW against a 100 mW part.

The chain is placed as a tight vertical run up the left edge, R10 to R33 to
R34, 1.9 mm apart. Spreading series resistors out would carry 40-80 V across
the board and couple noise into the divider midpoint; the first attempt
anchored R34 to R11 and produced a 14.5 mm run, now 2.4 mm.

The two new midpoints are at 80.7 V and 42.4 V. IPC-2221B wants 0.13 mm for
those with a coating and the board default of 0.15 mm already passes, but
1.15x is not much for 80 V, so a rule holds them at 0.25 mm and the pours
back off accordingly.

Also reverted: a "fix" to the START debounce capacitor that fixed nothing.
V1.3 wires U1.35 to START1 pin 1 and C13 to pin 2, which looked inconsistent
with the other three buttons. I read that as the capacitor filtering behind
the switch's contact resistance. It is not — the TS-1187A bonds pins 1 and 2
inside the package, and 3 and 4 likewise, with the moving contact between
the two pairs. The netlist says as much: START1.3 and START1.4 both go to
GND. C13 and U1.35 are already on one solid node. Changing it only added
7.4 mm of track.

Netlist verifies at 229 connections against V1.3 plus the declared changes.
ERC and DRC both clean.

Co-Authored-By: Claude Opus 5 <noreply@anthropic.com>
Parts:
- added R33: 115k, R0603, F.Cu at (122.5, 87.4)
- added R34: 115k, R0603, F.Cu at (122.4, 85.5)
- R10: value (none) -> 118k
Connections:
- R10 pad 1: VOUT_SENSE -> HV_DIV1
Routing:
- net VOUT_SENSE: track 6.74 -> 13.8 mm
- net HV_DIV2: track 0.00 -> 2.36 mm
- net HV_DIV1: track 0.00 -> 1.91 mm

Commit message: Move the ADS1115 back to 3.3 V and rescale the divider to suit
The I2C bus could not have worked reliably as drawn. The ADS1115 needs
0.7 x VDD to read a logic high — 3.50 V at a 5 V supply — while R5 and R6
pull the bus up to VDD33, so the high level is 3.3 V. Two tenths of a volt
below threshold, on a board that has not been built, so nothing has ever
exercised it. At 3.3 V the threshold drops to 2.31 V and the margin becomes
1.43x.

The reason it was at 5 V in the first place was range: V1.2 ran the part at
3.3 V and could not measure to 120 V. R11 covers that instead, 12k to
9.09k. At 120 V input AIN0 now reads 3.0547 V, inside the 3.6 V pin limit,
and the ceiling rises from 122.9 V to 141.4 V — at 5 V the PGA's 4.096 V
was the binding constraint, at 3.3 V it is the pin, and the pin is the more
generous of the two. Resolution goes from 3.750 to 4.910 mV per LSB, which
at 120 V is 0.004%.

Two consequences to carry into the firmware work:

- The divider coefficient changes from 30.000 to 39.284. This is exactly
  what the planned hw_info EEPROM is for — divider values that differ per
  hardware revision.
- CP shares this ADC through its own 150R/51R divider, so its measurement
  ceiling drops from 20.9 V to 14.2 V. Charging measured 8.99 V, leaving
  58% headroom, but if the TES spec permits 12 V that falls to 18%. Worth
  confirming against a real vehicle.

The R10 split also moves to Yageo's RT thin-film series rather than the
generic 1% parts I first used. The divider ratio *is* the voltage reading's
accuracy; three 1% resistors in the upper arm would take it from 0.1% to
about 0.58%. These part numbers follow the series' documented pattern but
need checking against LCSC stock — RT does not carry every E96 value.

Also fixed: _pcb_apply_nets ripped the tracks off any pad named in a
set_net, including ones already on the target net, which quietly
disconnected HV_DIV1 on the second run.

DRC and ERC clean, netlist 230 connections with zero difference, and all
fo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
Parts:
- R10: value 118k -> RT0603BRD07118KL
- R11: value (none) -> RT0603BRD079K09L
Connections:
- C20 pad 1: 5V -> VDD33
- U5 pad 8: 5V -> VDD33
Routing:
- net VDD33: track 86.7 -> 133.5 mm, vias 7 -> 9
- net 5V: track 61.3 -> 51.9 mm, vias 9 -> 7
- net HV_DIV1: track 1.91 -> 1.20 mm
