File: hardware/kicad/TES_Controller.kicad_sch (KiCad schematic)
At the start: 81 parts, among them CN1 B2PS-VH, CN2 S4B-XH-A, CN3 DG381-3.5-02P-14-00A, CN5 DG381-3.5-02P-14-00A, CN6 DG381-3.5-02P-14-00A, Q1 AO3400A, Q2 AO3400A, Q3 AO3400A, Q4 AO3401A, U1 ESP32-S3-WROOM-1, U10 DG301-5.0-02P-14-00A, U12 TJA1051T_3_1J, U5 ADS1115IDGSR, U6 AMS1117-3.3, U8 LMZM23601V5SILR

Commit message: Use one resistor value for the whole divider upper arm
Chris pointed out the upper arm could be three 115k rather than
118k + 115k + 115k. He is right, and my reason for the mixed values had
already expired: I picked them to sum to exactly 348k so the firmware
coefficient would not move, but moving the ADS1115 to 3.3 V changes R11 and
therefore the coefficient regardless. There was nothing left to preserve.

Every figure is effectively unchanged — 39.0 V per resistor against the same
1.9x margin, 4.869 vs 4.910 mV per LSB, a 140.2 V ceiling instead of 141.4 V
— and it drops a part number. That is not only the parts: JLCPCB charges a
setup fee per distinct component in SMT assembly.

Coefficient becomes 38.954, (345k + 9.09k) / 9.09k.

Also in this commit, recovering from something that has now happened twice:
KiCad was open on an old copy of the project the whole time we were working,
and on closing it wrote that copy back. The schematic lost all 8 components
added since (R33, R34, D9, D10, W1-W4) and the project file regained the
HV120 and Power netclasses along with a 0.2 mm clearance, which is where 534
DRC violations appeared from — against netclasses deleted days earlier. The
.kicad_dru was untouched, since KiCad does not rewrite it.

tools/check_project.py compares the settings that matter and regen_hw.sh
runs it before DRC, so the next occurrence is a one-line message rather than
a debugging session. The two .lck files were committed by accident and are
now untracked and ignored.

Co-Authored-By: Claude Opus 5 <noreply@anthropic.com>
Parts:
- R10: value RT0603BRD07118KL -> RT0603BRD07115KL
